File: eagle-stuffs/audio.brd (EAGLE design)
At the start: 57.1 x 44.5 mm, 20 parts, among them IC1 LM386N-1, IC2 TL084P, IC3 X9C102P, IC4 X9C102P

Commit message: Working on audio board
Parts:
- added C6: 0.01u, rcl:C025-025X050
- added R1: 10k, resistor:0207/10
- added U1: AT42QT1010SOT23, SparkFun-DigitalIC:SOT23-6
Connections:
- removed net N$15: CTRL.6, ROTARY.3
- removed net N$16: CTRL.8, ROTARY.4
- removed net N$17: CTRL.10, ROTARY.5
- new net VCC: U1.5
- net +5V: no longer ROTARY.1
- net GND: no longer ROTARY.2
Changed lines of the file:
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@@
 <layer number="48" name="Document" color="7" fill="1" visible="yes" active="yes"/>
 <layer number="49" name="Reference" color="7" fill="1" visible="yes" active="yes"/>
+<layer number="50" name="dxf" color="7" fill="1" visible="no" active="no"/>
 <layer number="51" name="tDocu" color="7" fill="1" visible="yes" active="yes"/>
 <layer number="52" name="bDocu" color="7" fill="1" visible="yes" active="yes"/>
+<layer number="53" name="tGND_GNDA" color="7" fill="9" visible="no" active="no"/>
+<layer number="54" name="bGND_GNDA" color="1" fill="9" visible="no" active="no"/>
+<layer number="56" name="wert" color="7" fill="1" visible="no" active="no"/>
+<layer number="90" name="Modules" color="5" fill="1" visible="no" active="no"/>
 <layer number="91" name="Nets" color="2" fill="1" visible="no" active="no"/>
 <layer number="92" name="Busses" color="1" fill="1" visible="no" active="no"/>
@@
 <layer number="98" name="Guide" color="6" fill="1" visible="no" active="no"/>
 <layer number="99" name="SpiceOrder" color="5" fill="1" visible="no" active="no"/>
+<layer number="100" name="Muster" color="7" fill="1" visible="no" active="no"/>
+<layer number="101" name="Patch_Top" color="12" fill="4" visible="yes" active="yes"/>
+<layer number="102" name="Vscore" color="7" fill="1" visible="yes" active="yes"/>
+<layer number="103" name="tMap" color="7" fill="1" visible="yes" active="yes"/>
+<layer number="104" name="Name" color="16" fill="1" visible="yes" active="yes"/>
+<layer number="105" name="tPlate" color="7" fill="1" visible="yes" active="yes"/>
+<layer number="106" name="bPlate" color="7" fill="1" visible="yes" active="yes"/>
+<layer number="107" name="Crop" color="7" fill="1" visible="yes" active="yes"/>
+<layer number="108" name="tplace-old" color="10" fill="1" visible="yes" active="yes"/>
+<layer number="109" name="ref-old" color="11" fill="1" visible="yes" active="yes"/>
+<layer number="116" name="Patch_BOT" color="9" fill="4" visible="yes" active="yes"/>
+<layer number="121" name="_tsilk" color="7" fill="1" visible="yes" active="yes"/>
+<layer number="122" name="_bsilk" color="7" fill="1" visible="yes" active="yes"/>
+<layer number="125" name="_tNames" color="7" fill="1" visible="yes" active="yes"/>
+<layer number="144" name="Drill_legend" color="7" fill="1" visible="yes" active="yes"/>
+<layer number="151" name="HeatSink" color="7" fill="1" visible="yes" active="yes"/>
+<layer number="199" name="Contour" color="7" fill="1" visible="yes" active="yes"/>
+<layer number="200" name="200bmp" color="1" fill="10" visible="yes" active="yes"/>
+<layer number="201" name="201bmp" color="2" fill="10" visible="yes" active="yes"/>
+<layer number="202" name="202bmp" color="3" fill="10" visible="yes" active="yes"/>
+<layer number="203" name="203bmp" color="4" fill="10" visible="yes" active="yes"/>
+<layer number="204" name="204bmp" color="5" fill="10" visible="yes" active="yes"/>
+<layer number="205" name="205bmp" color="6" fill="10" visible="yes" active="yes"/>
+<layer number="206" name="206bmp" color="7" fill="10" visible="yes" active="yes"/>
+<layer number="207" name="207bmp" color="8" fill="10" visible="yes" active="yes"/>
+<layer number="208" name="208bmp" color="9" fill="10" visible="yes" active="yes"/>
+<layer number="209" name="209bmp" color="7" fill="1" visible="yes" active="yes"/>
+<layer number="210" name="210bmp" color="7" fill="1" visible="yes" active="yes"/>
+<layer number="211" name="211bmp" color="7" fill="1" visible="yes" active="yes"/>
+<layer number="212" name="212bmp" color="7" fill="1" visible="yes" active="yes"/>
+<layer number="213" name="213bmp" color="7" fill="1" visible="yes" active="yes"/>
+<layer number="214" name="214bmp" color="7" fill="1" visible="yes" active="yes"/>
+<layer number="215" name="215bmp" color="7" fill="1" visible="yes" active="yes"/>
+<layer number="216" name="216bmp" color="7" fill="1" visible="yes" active="yes"/>
+<layer number="217" name="217bmp" color="18" fill="1" visible="no" active="no"/>
+<layer number="218" name="218bmp" color="19" fill="1" visible="no" active="no"/>
+<layer number="219" name="219bmp" color="20" fill="1" visible="no" active="no"/>
+<layer number="220" name="220bmp" color="21" fill="1" visible="no" active="no"/>
+<layer number="221" name="221bmp" color="22" fill="1" visible="no" active="no"/>
+<layer number="222" name="222bmp" color="23" fill="1" visible="no" active="no"/>
+<layer number="223" name="223bmp" color="24" fill="1" visible="no" active="no"/>
+<layer number="224" name="224bmp" color="25" fill="1" visible="no" active="no"/>
+<layer number="250" name="Descript" color="3" fill="1" visible="no" active="no"/>
+<layer number="251" name="SMDround" color="12" fill="11" visible="no" active="no"/>
+<layer number="254" name="cooling" color="7" fill="1" visible="yes" active="yes"/>
 </layers>
 <board>
@@
 <classes>
 <class number="0" name="default" width="0" drill="0">
+<clearance class="0" value="0.205"/>
 </class>
 </classes>
@@
 <element name="C5" library="rcl" package="E2,5-5" value="100uF" x="44.45" y="20.32"/>
 <element name="C2" library="rcl" package="C025-025X050" value="0.01u" x="44.45" y="13.97"/>
+<element name="U1" library="SparkFun-DigitalIC" package="SOT23-6" value="AT42QT1010SOT23" x="50.8" y="21.59"/>
+<element name="R1" library="resistor" package="0207/10" value="10k" x="6.35" y="-3.81"/>
+<element name="C6" library="rcl" package="C025-025X050" value="0.01u" x="3.81" y="-8.89"/>
 </elements>
 <signals>
@@
 <contactref element="MIC" pad="1"/>
 <contactref element="R6" pad="1"/>
-<contactref element="ROTARY" pad="2"/>
 <contactref element="IC2" pad="11"/>
 <contactref element="CTRL" pad="2"/>
 <contactref element="C5" pad="-"/>
-<wire x1="50.8" y1="26.67" x2="30.48" y2="38.1" width="0" layer="19" extent="1-1"/>
 <wire x1="45.72" y1="24.13" x2="50.8" y2="26.67" width="0" layer="19" extent="1-1"/>
+<wire x1="45.72" y1="20.32" x2="45.72" y2="24.13" width="0" layer="19" extent="1-1"/>
 <wire x1="40.64" y1="24.13" x2="45.72" y2="24.13" width="0" layer="19" extent="1-1"/>
-<wire x1="45.72" y1="20.32" x2="40.64" y2="24.13" width="0" layer="19" extent="1-1"/>
-<wire x1="30.48" y1="24.13" x2="45.72" y2="20.32" width="0" layer="19" extent="1-1"/>
+<wire x1="30.48" y1="24.13" x2="40.64" y2="24.13" width="0" layer="19" extent="1-1"/>
 <wire x1="21.59" y1="16.51" x2="30.48" y2="24.13" width="0" layer="19" extent="1-1"/>
 <wire x1="13.97" y1="24.13" x2="21.59" y2="16.51" width="0" layer="19" extent="1-1"/>
@@
 <wire x1="5.08" y1="10.16" x2="5.08" y2="16.51" width="0" layer="19" extent="1-1"/>
 <wire x1="27.94" y1="5.08" x2="21.59" y2="16.51" width="0" layer="19" extent="1-1"/>
-<wire x1="43.18" y1="5.08" x2="45.72" y2="20.32" width="0" layer="19" extent="1-1"/>
-<wire x1="7.62" y1="40.64" x2="13.97" y2="24.13" width="0" layer="19" extent="1-1"/>
-<wire x1="5.08" y1="38.1" x2="7.62" y2="40.64" width="0" layer="19" extent="1-1"/>
+<wire x1="30.48" y1="38.1" x2="30.48" y2="24.13" width="0" layer="19" extent="1-1"/>
+<wire x1="5.08" y1="38.1" x2="13.97" y2="24.13" width="0" layer="19" extent="1-1"/>
+<wire x1="7.62" y1="40.64" x2="5.08" y2="38.1" width="0" layer="19" extent="1-1"/>
 </signal>
 <signal name="N$2">
@@
 <contactref element="IC2" pad="4"/>
 <contactref element="CTRL" pad="4"/>
-<contactref element="ROTARY" pad="1"/>
 <contactref element="C5" pad="+"/>
-<wire x1="43.18" y1="31.75" x2="27.94" y2="38.1" width="0" layer="19" extent="1-1"/>
 <wire x1="43.18" y1="20.32" x2="43.18" y2="31.75" width="0" layer="19" extent="1-1"/>
 <wire x1="31.75" y1="20.32" x2="43.18" y2="20.32" width="0" layer="19" extent="1-1"/>
 <wire x1="27.94" y1="12.7" x2="31.75" y2="20.32" width="0" layer="19" extent="1-1"/>
 <wire x1="17.78" y1="5.08" x2="27.94" y2="12.7" width="0" layer="19" extent="1-1"/>
-<wire x1="40.64" y1="5.08" x2="43.18" y2="20.32" width="0" layer="19" extent="1-1"/>
 <wire x1="22.86" y1="31.75" x2="31.75" y2="20.32" width="0" layer="19" extent="1-1"/>
+<wire x1="27.94" y1="38.1" x2="22.86" y2="31.75" width="0" layer="19" extent="1-1"/>
 <wire x1="6.35" y1="31.75" x2="22.86" y2="31.75" width="0" layer="19" extent="1-1"/>
 </signal>
@@
 <wire x1="20.32" y1="12.7" x2="20.32" y2="40.64" width="0" layer="19" extent="1-1"/>
 </signal>
-<signal name="N$15">
-<contactref element="ROTARY" pad="3"/>
-<contactref element="CTRL" pad="6"/>
-<wire x1="45.72" y1="5.08" x2="25.4" y2="38.1" width="0" layer="19" extent="1-1"/>
-</signal>
-<signal name="N$16">
-<contactref element="ROTARY" pad="4"/>
-<contactref element="CTRL" pad="8"/>
-<wire x1="48.26" y1="5.08" x2="22.86" y2="38.1" width="0" layer="19" extent="1-1"/>
-</signal>
-<signal name="N$17">
-<contactref element="ROTARY" pad="5"/>
-<contactref element="CTRL" pad="10"/>
-<wire x1="50.8" y1="5.08" x2="20.32" y2="38.1" width="0" layer="19" extent="1-1"/>
-</signal>
 <signal name="N$5">
 <contactref element="C2" pad="2"/>
@@
 <wire x1="45.72" y1="13.97" x2="43.18" y2="24.13" width="0" layer="19" extent="1-1"/>
 </signal>
+<signal name="VCC">
+<contactref element="U1" pad="5"/>
+</signal>
 </signals>

Commit message: Still working on audio…
Parts:
- removed ROTARY: (no value), pinhead:1X05
- added C7: 1, rcl:C025-025X050
- added C8: 2.2nF, rcl:C025-025X050
- added R8: 100K, resistor:0207/10
- added R9: 33K, resistor:0207/10
- added SPK1: (no value), pinhead:1X02
- C4: value 0.1u -> 0.1
- C6: value 0.01u -> 10nF
- IC3, IC4: value X9C102P -> DS1804
- R5: value 7K -> 10K
- R6: value 3K -> 15K
- moved C6 50.6 mm to (49.5, 12.7)
- moved R1 40.6 mm to (44.5, 10.2)
Connections:
- removed net VCC: U1.5
- new net N$15: C7.1, IC2.3, R4.2, R8.1
- new net N$16: C6.1, R1.2, U1.3
- new net N$17: C6.2, U1.4
- new net N$22: R1.1, SPK1.1
- new net N$24: CTRL.6, U1.1
- new net N$8: C4.2, R7.2
- net +5V: now also R8.2, U1.5, U1.6
- net GND: now also C7.2, C8.2, U1.2; no longer R7.1
- net N$10: now also IC2.2, IC4.3, IC4.5, R7.1; no longer C4.2, IC2.3, R4.2
- net N$11: now also IC4.6, R9.2; no longer IC2.5, IC4.3
- net N$13: now also C8.1, IC2.5, R9.1; no longer IC2.2, IC4.5, R7.2

Commit message: Found SSM2211 lib… still going
Parts:
- removed IC1: LM386N-1, linear:DIL08
- added U2: SSM2211SZ, Analog Devices_By_element14_Batch_1:SOIC127P600X175-8N
Connections:
- removed net N$2: C2.1, IC3.5
- removed net N$3: C3.2, R2.2
- removed net N$4: C1.+, C3.1, IC1.5
- removed net N$5: C2.2, IC1.3
- removed net N$6: IC1.1
- removed net N$7: C1.-, SPK.1
- new net V+: U2.6
- new net V-: U2.7
- new net VCC: IC3.8
- net +5V: no longer C5.+, IC1.6, IC3.8
- net GND: no longer C5.-, IC1.2, IC1.4, R2.1
- net N$1: now also IC3.5; no longer IC3.6, IN.2
Changed lines of the file:
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@@
 </autorouter>
 <elements>
-<element name="IC1" library="linear" package="DIL08" value="LM386N-1" x="41.91" y="27.94" smashed="yes">
-<attribute name="NAME" x="36.576" y="25.019" size="1.27" layer="25" ratio="10" rot="R90"/>
-<attribute name="VALUE" x="38.354" y="27.305" size="1.27" layer="27" ratio="10"/>
-</element>
 <element name="IC2" library="linear" package="DIL14" value="TL084P" x="27.94" y="8.89" smashed="yes" rot="R180">
 <attribute name="NAME" x="37.211" y="11.938" size="1.27" layer="25" ratio="10" rot="R270"/>
@@
 <element name="C8" library="rcl" package="C025-025X050" value="2.2nF" x="54.61" y="33.02"/>
 <element name="SPK1" library="pinhead" package="1X02" value="" x="45.72" y="5.08"/>
+<element name="U2" library="Analog Devices_By_element14_Batch_1" package="SOIC127P600X175-8N" value="SSM2211SZ" x="40.64" y="27.94">
+<attribute name="PACKAGE" value="SOIC-8" x="40.64" y="27.94" size="1.778" layer="27" display="off"/>
+<attribute name="OC_NEWARK" value="19M1049" x="40.64" y="27.94" size="1.778" layer="27" display="off"/>
+<attribute name="MPN" value="SSM2211SZ" x="40.64" y="27.94" size="1.778" layer="27" display="off"/>
+<attribute name="SUPPLIER" value="Analog Devices" x="40.64" y="27.94" size="1.778" layer="27" display="off"/>
+<attribute name="OC_FARNELL" value="9994440" x="40.64" y="27.94" size="1.778" layer="27" display="off"/>
+</element>
 </elements>
 <signals>
 <signal name="GND">
-<contactref element="IC1" pad="4"/>
-<contactref element="IC3" pad="4"/>
-<contactref element="IC1" pad="2"/>
-<contactref element="R2" pad="1"/>
 <contactref element="SPK" pad="2"/>
 <contactref element="IN" pad="1"/>
 <contactref element="IC2" pad="11"/>
 <contactref element="CTRL" pad="2"/>
-<contactref element="C5" pad="-"/>
 <contactref element="MIC" pad="1"/>
 <contactref element="R4" pad="1"/>
@@
 <contactref element="U1" pad="2"/>
 <contactref element="IC4" pad="4"/>
-<wire x1="45.72" y1="24.13" x2="50.8" y2="26.67" width="0" layer="19" extent="1-1"/>
-<wire x1="45.72" y1="20.32" x2="45.72" y2="24.13" width="0" layer="19" extent="1-1"/>
-<wire x1="50.8" y1="20.2149" x2="45.72" y2="20.32" width="0" layer="19" extent="1-1"/>
-<wire x1="40.64" y1="24.13" x2="45.72" y2="24.13" width="0" layer="19" extent="1-1"/>
-<wire x1="30.48" y1="24.13" x2="40.64" y2="24.13" width="0" layer="19" extent="1-1"/>
+<contactref element="IC3" pad="4"/>
+<wire x1="50.8" y1="26.67" x2="55.88" y2="33.02" width="0" layer="19" extent="1-1"/>
+<wire x1="50.8" y1="20.2149" x2="50.8" y2="26.67" width="0" layer="19" extent="1-1"/>
+<wire x1="38.1" y1="21.59" x2="50.8" y2="20.2149" width="0" layer="19" extent="1-1"/>
+<wire x1="30.48" y1="24.13" x2="38.1" y2="21.59" width="0" layer="19" extent="1-1"/>
 <wire x1="30.48" y1="38.1" x2="30.48" y2="24.13" width="0" layer="19" extent="1-1"/>
 <wire x1="13.97" y1="24.13" x2="30.48" y2="24.13" width="0" layer="19" extent="1-1"/>
@@
 <wire x1="5.08" y1="10.16" x2="5.08" y2="16.51" width="0" layer="19" extent="1-1"/>
 <wire x1="5.08" y1="38.1" x2="13.97" y2="24.13" width="0" layer="19" extent="1-1"/>
-<wire x1="7.62" y1="40.64" x2="5.08" y2="38.1" width="0" layer="19" extent="1-1"/>
-<wire x1="38.1" y1="21.59" x2="5.08" y2="10.16" width="0" layer="19" extent="1-1"/>
-<wire x1="55.88" y1="33.02" x2="38.1" y2="21.59" width="0" layer="19" extent="1-1"/>
 <wire x1="27.94" y1="5.08" x2="30.48" y2="24.13" width="0" layer="19" extent="1-1"/>
 </signal>
-<signal name="N$2">
-<contactref element="IC3" pad="5"/>
-<contactref element="C2" pad="1"/>
-<wire x1="13.97" y1="31.75" x2="43.18" y2="13.97" width="0" layer="19" extent="1-1"/>
-</signal>
-<signal name="N$1">
-<contactref element="IC3" pad="6"/>
-<contactref element="IN" pad="2"/>
-<wire x1="5.08" y1="35.56" x2="11.43" y2="31.75" width="0" layer="19" extent="1-1"/>
-</signal>
 <signal name="+5V">
-<contactref element="IC1" pad="6"/>
-<contactref element="IC3" pad="8"/>
 <contactref element="R3" pad="2"/>
 <contactref element="IC2" pad="4"/>
 <contactref element="CTRL" pad="4"/>
-<contactref element="C5" pad="+"/>
 <contactref element="U1" pad="5"/>
 <contactref element="U1" pad="6"/>
@@
 <contactref element="IC4" pad="8"/>
 <contactref element="R5" pad="2"/>
-<wire x1="49.85" y1="22.9651" x2="43.18" y2="31.75" width="0" layer="19" extent="1-1"/>
+<wire x1="49.85" y1="22.9651" x2="44.45" y2="34.29" width="0" layer="19" extent="1-1"/>
 <wire x1="50.8" y1="22.9651" x2="49.85" y2="22.9651" width="0" layer="19" extent="1-1"/>
-<wire x1="43.18" y1="20.32" x2="49.85" y2="22.9651" width="0" layer="19" extent="1-1"/>
-<wire x1="31.75" y1="20.32" x2="43.18" y2="20.32" width="0" layer="19" extent="1-1"/>
+<wire x1="27.94" y1="38.1" x2="44.45" y2="34.29" width="0" layer="19" extent="1-1"/>
+<wire x1="22.86" y1="31.75" x2="27.94" y2="38.1" width="0" layer="19" extent="1-1"/>
+<wire x1="31.75" y1="20.32" x2="22.86" y2="31.75" width="0" layer="19" extent="1-1"/>
 <wire x1="27.94" y1="12.7" x2="31.75" y2="20.32" width="0" layer="19" extent="1-1"/>
 <wire x1="17.78" y1="5.08" x2="27.94" y2="12.7" width="0" layer="19" extent="1-1"/>
-<wire x1="44.45" y1="34.29" x2="17.78" y2="5.08" width="0" layer="19" extent="1-1"/>
-<wire x1="22.86" y1="31.75" x2="31.75" y2="20.32" width="0" layer="19" extent="1-1"/>
-<wire x1="27.94" y1="38.1" x2="22.86" y2="31.75" width="0" layer="19" extent="1-1"/>
-<wire x1="6.35" y1="31.75" x2="22.86" y2="31.75" width="0" layer="19" extent="1-1"/>
-</signal>
-<signal name="N$3">
-<contactref element="C3" pad="2"/>
-<contactref element="R2" pad="2"/>
-<wire x1="17.78" y1="40.64" x2="41.91" y2="38.1" width="0" layer="19" extent="1-1"/>
-</signal>
-<signal name="N$4">
-<contactref element="IC1" pad="5"/>
-<contactref element="C1" pad="+"/>
-<contactref element="C3" pad="1"/>
-<wire x1="48.514" y1="38.1" x2="45.72" y2="31.75" width="0" layer="19" extent="1-1"/>
-<wire x1="39.37" y1="38.1" x2="48.514" y2="38.1" width="0" layer="19" extent="1-1"/>
-</signal>
-<signal name="N$6">
-<contactref element="IC1" pad="1"/>
-</signal>
-<signal name="N$7">
-<contactref element="C1" pad="-"/>
-<contactref element="SPK" pad="1"/>
-<wire x1="50.546" y1="38.1" x2="50.8" y2="29.21" width="0" layer="19" extent="1-1"/>
 </signal>
 <signal name="N$9">
@@
 <contactref element="IC2" pad="7"/>
 <wire x1="20.32" y1="12.7" x2="20.32" y2="40.64" width="0" layer="19" extent="1-1"/>
-</signal>
-<signal name="N$5">
-<contactref element="C2" pad="2"/>
-<contactref element="IC1" pad="3"/>
-<wire x1="45.72" y1="13.97" x2="43.18" y2="24.13" width="0" layer="19" extent="1-1"/>
 </signal>
 <signal name="N$8">
@@
 <wire x1="44.45" y1="5.08" x2="39.37" y2="10.16" width="0" layer="19" extent="1-1"/>
 </signal>
+<signal name="V+">
+<contactref element="U2" pad="6"/>
+</signal>
+<signal name="V-">
+<contactref element="U2" pad="7"/>
+</signal>
+<signal name="N$1">
+<contactref element="IC3" pad="5"/>
+</signal>
+<signal name="VCC">
+<contactref element="IC3" pad="8"/>
+</signal>
 </signals>

Commit message: This should work…
Parts:
- removed C8: 2.2nF, rcl:C025-025X050
- removed SPK1: (no value), pinhead:1X02
- added R10: 10K, resistor:0207/10
- added TOUCH: (no value), adafruit:1X01
- C2: value 0.01u -> 2.2
- C3: value 0.047u -> 2.2
- C5: value 100uF -> 1; device rcl:E2,5-5 -> rcl:C025-025X050
- C6: value 10nF -> 2.2nF
- C7: value 1 -> 10nF
- IC3: value DS1804 -> DS1804-10k
- R2: value 10 -> 8k
- R3: value 10K -> 10k
- R4: value 100K -> 15K
- R6: value 15K -> 33K
- R9: value 33K -> 100K
- moved R6 37.4 mm to (45.7, 8.89)
- moved C5 35.2 mm to (12.7, 5.08)
- moved R3 31.2 mm to (26.7, 33.0)
- moved R1 30.5 mm to (43.2, 40.6)
- moved C7 22.6 mm to (50.8, 39.4), turned to 270 degrees
- moved R5 20.5 mm to (45.7, 12.7)
- moved R7 19.0 mm to (45.7, 16.5)
- moved R8 18.9 mm to (33.0, 16.5)
- moved IC4 18.0 mm to (8.89, 25.4)
- moved R9 17.8 mm to (20.3, 16.5)
- moved IC3 16.7 mm to (26.7, 25.4)
- moved U1 14.9 mm to (45.7, 35.6), turned to 180 degrees
- moved C6 11.7 mm to (40.6, 5.08)
- moved C1 9.67 mm to (45.7, 29.2)
- moved C2 9.16 mm to (39.4, 21.6)
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Connections:
- removed net V+: U2.6
- removed net V-: U2.7
- new net N$2: C2.1, IN.2
- new net N$3: C2.2, R3.2
- new net N$4: R2.2, R3.1, U2.4
- new net N$5: C3.1, U2.2, U2.3
- new net N$6: SPK.1, U2.8
- new net N$7: IC3.5, IC3.6, R2.1
- net +5V: now also C1.+, IC3.8, R10.2, U2.6; no longer R3.2
- net GND: now also C1.-, C3.2, C5.2, C6.2, R9.1, U2.7; no longer C7.2, C8.2, R6.1, SPK.2
- net N$1: now also IC3.3, SPK.2, U2.5; no longer IC3.5
- net N$11: now also R6.2; no longer R9.2
- net N$12: now also R4.2; no longer R6.2
- net N$13: now also C6.1, R6.1; no longer C8.1, R9.1
- net N$15: now also C5.1, R9.2; no longer C7.1, R4.2
- net N$16: now also C7.1; no longer C6.1
- net N$17: now also C7.2; no longer C6.2
- net N$22: now also TOUCH.1; no longer SPK1.1
- net N$9: now also R10.1; no longer R3.1
- net VCC: now also CTRL.8, U2.1; no longer IC3.8
Routing:
- net GND: track 0.00 -> 180.9 mm
- net +5V: track 0.00 -> 137.4 mm
- net N$20: track 0.00 -> 64.9 mm
- net N$11: track 0.00 -> 62.3 mm
- net N$10: track 0.00 -> 57.6 mm
- net N$14: track 0.00 -> 55.4 mm
- net N$21: track 0.00 -> 42.4 mm
- net N$2: track 0.00 -> 40.0 mm
- net N$8: track 0.00 -> 40.0 mm
- net N$1: track 0.00 -> 32.0 mm
- net N$12: track 0.00 -> 31.0 mm
- net VCC: track 0.00 -> 28.2 mm
- net N$15: track 0.00 -> 27.0 mm
- net N$19: track 0.00 -> 26.4 mm
- net N$4: track 0.00 -> 25.0 mm
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Other:
- board text removed: "Rev. A"

Commit message: Waiting for proto board test design
Parts:
- added C8: 0.1, rcl:C025-025X050
- C4: value 0.1 -> 1
- C7: value 10nF -> 0.01
- R10: value 10K -> 1k
- moved C6 7.62 mm to (48.3, 5.08)
- moved C3 6.35 mm to (35.6, 30.5)
- moved C7 6.35 mm to (45.7, 35.6)
- moved U2 5.39 mm to (35.6, 25.4)
- moved C1 4.58 mm to (43.2, 25.4)
- moved SPK 4.58 mm to (52.1, 25.4)
- moved C2 4.02 mm to (35.6, 20.3)
- moved TOUCH 3.81 mm to (35.6, 36.8), turned to 90 degrees
- moved U1 3.81 mm to (49.5, 35.6)
- moved IC3 2.54 mm to (24.1, 25.4)
- moved R3 2.54 mm to (24.1, 33.0)
- moved R1 2.54 mm to (40.6, 40.6)
- moved R2 2.54 mm to (10.2, 33.0)
- moved R5 2.54 mm to (48.3, 12.7)
- moved R6 2.54 mm to (48.3, 8.89)
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Connections:
- net +5V: now also C8.1
- net GND: now also C8.2
- net N$10: no longer IC4.3
- net N$7: no longer IC3.6
Routing:
- net GND: track 180.9 -> 0.00 mm
- net +5V: track 137.4 -> 0.00 mm
- net N$20: track 64.9 -> 0.00 mm
- net N$11: track 62.3 -> 0.00 mm
- net N$10: track 57.6 -> 0.00 mm
- net N$14: track 55.4 -> 0.00 mm
- net N$21: track 42.4 -> 0.00 mm
- net N$2: track 40.0 -> 0.00 mm
- net N$8: track 40.0 -> 0.00 mm
- net N$1: track 32.0 -> 0.00 mm
- net N$12: track 31.0 -> 0.00 mm
- net VCC: track 28.2 -> 0.00 mm
- net N$15: track 27.0 -> 0.00 mm
- net N$19: track 26.4 -> 0.00 mm
- net N$4: track 25.0 -> 0.00 mm
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