File: eagle-stuffs/audio.brd (EAGLE design)
At the start: 57.1 x 44.5 mm, 35 parts, among them IC1 SSM2211SZ, IC2 TL084P, IC4 DS1804-10k

Commit message: Change R13 value
Going at 10k on the digit pot will have the reverse effect on gain and
shutdown the mic.
Parts:
- R13: value 5.1k -> 4.7k
Changed lines of the file:
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@@
 <element name="R8" library="rcl" package="0204V" value="10k" x="33.02" y="13.97"/>
 <element name="R12" library="rcl" package="0204V" value="15k" x="11.43" y="22.86"/>
-<element name="R13" library="rcl" package="0204V" value="5.1k" x="16.51" y="22.86"/>
+<element name="R13" library="rcl" package="0204V" value="4.7k" x="16.51" y="22.86"/>
 <element name="R9" library="rcl" package="0204V" value="1k" x="26.67" y="22.86"/>
 <element name="C1" library="rcl" package="E3,5-10" value="220" x="48.26" y="36.83" smashed="yes">
