File: eagle-stuffs/lamp_board_simple.sch (EAGLE design)
At the start: 7 parts

Commit message: Ajustements to silk
Other:
- note added: "A"
Changed lines of the file:
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@@
 <text x="208.28" y="33.02" size="2.54" layer="98" font="fixed">Y.A.N.C. (Yet Another Nixie Clock)</text>
 <text x="190.5" y="15.24" size="2.54" layer="98" font="fixed">Licensed under CERN OHL v.1.2 or later</text>
+<text x="279.4" y="15.24" size="2.54" layer="98" font="fixed">A</text>
 </plain>
 <instances>

Commit message: Minor ajustements
Other:
- note added: "Note that those pinhead connector are mounted on the bottom layer. This is why the cathod connector on the driver board is mirror to account for this."
Changed lines of the file:
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@@
 <text x="190.5" y="15.24" size="2.54" layer="98" font="fixed">Licensed under CERN OHL v.1.2 or later</text>
 <text x="279.4" y="15.24" size="2.54" layer="98" font="fixed">A</text>
+<text x="129.54" y="187.96" size="2.54" layer="98" font="fixed">Note that those pinhead connector are
+mounted on the bottom layer.
+This is why the cathod connector on the
+driver board is mirror to account for this.</text>
 </plain>
 <instances>
@@
 </schematic>
 </drawing>
+<compatibility>
+<note version="6.3" minversion="6.2.2" severity="warning">
+Since Version 6.2.2 text objects can contain more than one line,
+which will not be processed correctly with this version.
+</note>
+</compatibility>
 </eagle>

Commit message: Corrected mirror pinout on nixie
Other:
- note added: "B"
- note removed: "A"
Changed lines of the file:
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@@
 <text x="208.28" y="33.02" size="2.54" layer="98" font="fixed">Y.A.N.C. (Yet Another Nixie Clock)</text>
 <text x="190.5" y="15.24" size="2.54" layer="98" font="fixed">Licensed under CERN OHL v.1.2 or later</text>
-<text x="279.4" y="15.24" size="2.54" layer="98" font="fixed">A</text>
+<text x="279.4" y="15.24" size="2.54" layer="98" font="fixed">B</text>
 <text x="129.54" y="187.96" size="2.54" layer="98" font="fixed">Note that those pinhead connector are
 mounted on the bottom layer.
@@
 <junction x="124.46" y="137.16"/>
 <wire x1="165.1" y1="177.8" x2="124.46" y2="177.8" width="0.1524" layer="91"/>
-<wire x1="124.46" y1="177.8" x2="124.46" y2="137.16" width="0.1524" layer="91"/>
 <pinref part="IN/OUT" gate="A" pin="1"/>
 <pinref part="OUT/IN" gate="A" pin="1"/>
+<wire x1="124.46" y1="177.8" x2="124.46" y2="137.16" width="0.1524" layer="91"/>
 </segment>
 </net>

Commit message: Added some info
Other:
- note added: "Nixies are mounted on top layer so connectors has been mirror on the board to account for this; otherwise wrong digit will lit up."
Changed lines of the file:
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@@
 This is why the cathod connector on the
 driver board is mirror to account for this.</text>
+<text x="78.74" y="48.26" size="2.54" layer="98" font="fixed">Nixies are mounted on top layer so
+connectors has been mirror on the board
+to account for this; otherwise
+wrong digit will lit up.</text>
 </plain>
 <instances>
