File: eagle-stuffs/audio.sch (EAGLE design)
At the start: 20 parts, among them IC1 LM386N-1, IC2 TL084P, IC3 X9C102P, IC4 X9C102P

Commit message: Working on audio board
Parts:
- added C6: 0.01u, rcl:C-US025-025X050
- added R1: 10k, resistor:R-US_0207/10
- added U1: AT42QT1010SOT23, SparkFun-DigitalIC:AT42QT1010SOT23
Connections:
- removed net N$15: CTRL.6, ROTARY.3
- removed net N$16: CTRL.8, ROTARY.4
- removed net N$17: CTRL.10, ROTARY.5
- new net VCC: U1.VDD
- net +5V: no longer ROTARY.1
- net GND: no longer ROTARY.2
Other:
- note added: "Author:"
- note added: "Licensed under CERN OHL v.1.2 or later"
- note added: "Project:"
- note added: "Steve Sirois"
- note added: "Y.A.N.C. (Yet Another Nixie Clock)"
- moved on the sheet: C1, C2, C3, C4, C5, CTRL, IC1, IC2A, IC2B, IC3, IC4, IN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

Commit message: Still working on audio…
Parts:
- removed ROTARY: (no value), pinhead:PINHD-1X5
- added C7: 1, rcl:C-US025-025X050
- added C8: 2.2nF, rcl:C-US025-025X050
- added R8: 100K, resistor:R-US_0207/10
- added R9: 33K, resistor:R-US_0207/10
- added SPK1: (no value), pinhead:PINHD-1X2
- C4: value 0.1u -> 0.1
- C6: value 0.01u -> 10nF
- IC3, IC4: value X9C102P -> DS1804
- R5: value 7K -> 10K
- R6: value 3K -> 15K
Connections:
- removed net VCC: U1.VDD
- new net N$15: C7.1, IC2A.+IN, R4.2, R8.1
- new net N$16: C6.1, R1.2, U1.SNSK
- new net N$17: C6.2, U1.SNS
- new net N$22: R1.1, SPK1.1
- new net N$24: CTRL.6, U1.OUT
- new net N$8: C4.2, R7.2
- net +5V: now also R8.2, U1.SYNC/MODE, U1.VDD
- net GND: now also C7.2, C8.2, U1.VSS; no longer R7.1
- net N$10: now also IC2A.-IN, IC4.H, IC4.W, R7.1; no longer C4.2, IC2A.+IN, R4.2
- net N$11: now also IC4.L, R9.2; no longer IC2B.+IN, IC4.H
- net N$13: now also C8.1, IC2B.+IN, R9.1; no longer IC2A.-IN, IC4.W, R7.2
Other:
- moved on the sheet: C4, C6, IC2A, IC2B, IC4, IN, MIC, R1, R3, R4, R5, R6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

Commit message: Found SSM2211 lib… still going
Parts:
- removed IC1: LM386N-1, linear:LM386N-1
- added U2: SSM2211SZ, Analog Devices_By_element14_Batch_1:SSM2211SZ
Connections:
- removed net N$2: C2.1, IC3.W
- removed net N$3: C3.2, R2.2
- removed net N$4: C1.+, C3.1, IC1.OUT
- removed net N$5: C2.2, IC1.+IN
- removed net N$6: IC1.GAIN@1
- removed net N$7: C1.-, SPK.1
- net +5V: no longer C5.+, IC1.VS, IC3.VCC
- net GND: no longer C5.-, IC1.-IN, IC1.GND, IC3.GND, R2.1
- net N$1: now also IC3.W; no longer IC3.L, IN.2
Other:
- moved on the sheet: C1, C2, C3, C5, R2
Changed lines of the file:
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@@
 <parts>
 <part name="FRAME1" library="frames" deviceset="FRAME_A_L" device=""/>
-<part name="IC1" library="linear" deviceset="LM386?-*" device="N" technology="1"/>
 <part name="IC2" library="linear" deviceset="TL084" device="P"/>
 <part name="IC3" library="pot-xicor" deviceset="X9C102*" device="P" value="DS1804"/>
@@
 <part name="C3" library="rcl" deviceset="C-US" device="025-025X050" value="0.047u"/>
 <part name="C4" library="rcl" deviceset="C-US" device="025-025X050" value="0.1"/>
-<part name="SUPPLY3" library="supply2" deviceset="GND" device=""/>
 <part name="SUPPLY4" library="supply2" deviceset="+5V" device=""/>
 <part name="SUPPLY5" library="supply2" deviceset="GND" device=""/>
@@
 <part name="SUPPLY13" library="supply2" deviceset="GND" device=""/>
 <part name="SPK1" library="pinhead" deviceset="PINHD-1X2" device=""/>
+<part name="U2" library="Analog Devices_By_element14_Batch_1" deviceset="SSM2211SZ" device=""/>
 </parts>
 <sheets>
@@
 <instance part="FRAME1" gate="G$1" x="0" y="0"/>
 <instance part="FRAME1" gate="G$2" x="172.72" y="0"/>
-<instance part="IC1" gate="G$1" x="142.24" y="182.88" smashed="yes">
-<attribute name="NAME" x="137.16" y="190.5" size="1.778" layer="95" rot="R180"/>
-<attribute name="VALUE" x="147.32" y="179.07" size="1.778" layer="96"/>
-</instance>
 <instance part="IC2" gate="A" x="83.82" y="50.8"/>
 <instance part="IC2" gate="B" x="142.24" y="48.26"/>
 <instance part="IC3" gate="1" x="83.82" y="170.18" rot="MR0"/>
 <instance part="IC4" gate="1" x="91.44" y="83.82" rot="MR0"/>
-<instance part="R2" gate="G$1" x="172.72" y="167.64" rot="R90"/>
+<instance part="R2" gate="G$1" x="226.06" y="182.88" rot="R90"/>
 <instance part="R3" gate="G$1" x="33.02" y="60.96" rot="R90"/>
 <instance part="R4" gate="G$1" x="58.42" y="38.1" rot="R90"/>
@@
 <instance part="SPK" gate="G$1" x="254" y="180.34"/>
 <instance part="IN" gate="G$1" x="20.32" y="165.1" rot="R180"/>
-<instance part="C1" gate="G$1" x="185.42" y="182.88" rot="R90"/>
-<instance part="C3" gate="G$1" x="172.72" y="177.8"/>
+<instance part="C1" gate="G$1" x="218.44" y="182.88" rot="R180"/>
+<instance part="C3" gate="G$1" x="200.66" y="182.88"/>
 <instance part="C4" gate="G$1" x="38.1" y="48.26" rot="R90"/>
-<instance part="SUPPLY3" gate="GND" x="129.54" y="157.48"/>
 <instance part="SUPPLY4" gate="+5V" x="139.7" y="205.74" smashed="yes">
 <attribute name="VALUE" x="137.795" y="208.915" size="1.778" layer="96"/>
@@
 <instance part="SUPPLY12" gate="GND" x="157.48" y="10.16"/>
 <instance part="CTRL" gate="A" x="236.22" y="139.7"/>
-<instance part="C5" gate="G$1" x="129.54" y="195.58" smashed="yes">
-<attribute name="NAME" x="123.063" y="196.0626" size="1.778" layer="95"/>
-<attribute name="VALUE" x="120.523" y="190.9826" size="1.778" layer="96"/>
+<instance part="C5" gate="G$1" x="193.04" y="182.88" smashed="yes">
+<attribute name="NAME" x="186.563" y="183.3626" size="1.778" layer="95"/>
+<attribute name="VALUE" x="184.023" y="178.2826" size="1.778" layer="96"/>
 </instance>
-<instance part="C2" gate="G$1" x="111.76" y="185.42" smashed="yes" rot="R90">
-<attribute name="NAME" x="111.125" y="186.436" size="1.778" layer="95" rot="R90"/>
-<attribute name="VALUE" x="115.951" y="186.436" size="1.778" layer="96" rot="R90"/>
+<instance part="C2" gate="G$1" x="172.72" y="182.88" smashed="yes">
+<attribute name="NAME" x="173.736" y="183.515" size="1.778" layer="95"/>
+<attribute name="VALUE" x="173.736" y="178.689" size="1.778" layer="96"/>
 </instance>
 <instance part="U1" gate="G$1" x="195.58" y="83.82"/>
@@
 <instance part="SUPPLY13" gate="GND" x="177.8" y="60.96"/>
 <instance part="SPK1" gate="G$1" x="259.08" y="86.36"/>
+<instance part="U2" gate="A" x="139.7" y="185.42"/>
 </instances>
 <busses>
 </busses>
 <nets>
-<net name="N$2" class="0">
-<segment>
-<pinref part="IC3" gate="1" pin="W"/>
-<wire x1="71.12" y1="170.18" x2="66.04" y2="170.18" width="0.1524" layer="91"/>
-<wire x1="66.04" y1="170.18" x2="66.04" y2="185.42" width="0.1524" layer="91"/>
-<pinref part="C2" gate="G$1" pin="1"/>
-<wire x1="66.04" y1="185.42" x2="109.22" y2="185.42" width="0.1524" layer="91"/>
-</segment>
-</net>
-<net name="N$1" class="0">
-<segment>
-<pinref part="IC3" gate="1" pin="L"/>
-<pinref part="IN" gate="G$1" pin="2"/>
-<wire x1="71.12" y1="165.1" x2="22.86" y2="165.1" width="0.1524" layer="91"/>
-</segment>
-</net>
 <net name="GND" class="0">
-<segment>
-<pinref part="IC1" gate="G$1" pin="GND"/>
-<pinref part="SUPPLY3" gate="GND" pin="GND"/>
-<wire x1="139.7" y1="175.26" x2="129.54" y2="175.26" width="0.1524" layer="91"/>
-<wire x1="129.54" y1="175.26" x2="129.54" y2="162.56" width="0.1524" layer="91"/>
-<pinref part="IC1" gate="G$1" pin="-IN"/>
-<wire x1="129.54" y1="162.56" x2="129.54" y2="160.02" width="0.1524" layer="91"/>
-<wire x1="134.62" y1="180.34" x2="129.54" y2="180.34" width="0.1524" layer="91"/>
-<wire x1="129.54" y1="180.34" x2="129.54" y2="175.26" width="0.1524" layer="91"/>
-<junction x="129.54" y="175.26"/>
-<pinref part="R2" gate="G$1" pin="1"/>
-<wire x1="172.72" y1="162.56" x2="129.54" y2="162.56" width="0.1524" layer="91"/>
-<junction x="129.54" y="162.56"/>
-<pinref part="IC3" gate="1" pin="GND"/>
-<wire x1="96.52" y1="162.56" x2="129.54" y2="162.56" width="0.1524" layer="91"/>
-<pinref part="C5" gate="G$1" pin="-"/>
-<wire x1="129.54" y1="190.5" x2="129.54" y2="180.34" width="0.1524" layer="91"/>
-<junction x="129.54" y="180.34"/>
-</segment>
 <segment>
 <pinref part="SPK" gate="G$1" pin="2"/>
@@
 <net name="+5V" class="0">
 <segment>
-<pinref part="IC1" gate="G$1" pin="VS"/>
-<pinref part="SUPPLY4" gate="+5V" pin="+5V"/>
-<wire x1="139.7" y1="190.5" x2="139.7" y2="198.12" width="0.1524" layer="91"/>
-<pinref part="IC3" gate="1" pin="VCC"/>
-<wire x1="139.7" y1="198.12" x2="139.7" y2="203.2" width="0.1524" layer="91"/>
-<wire x1="96.52" y1="177.8" x2="104.14" y2="177.8" width="0.1524" layer="91"/>
-<wire x1="104.14" y1="177.8" x2="104.14" y2="198.12" width="0.1524" layer="91"/>
-<wire x1="104.14" y1="198.12" x2="129.54" y2="198.12" width="0.1524" layer="91"/>
-<junction x="139.7" y="198.12"/>
-<pinref part="C5" gate="G$1" pin="+"/>
-<wire x1="129.54" y1="198.12" x2="139.7" y2="198.12" width="0.1524" layer="91"/>
-<junction x="129.54" y="198.12"/>
-</segment>
-<segment>
 <pinref part="R3" gate="G$1" pin="2"/>
 <pinref part="SUPPLY7" gate="+5V" pin="+5V"/>
@@
 </segment>
 </net>
-<net name="N$3" class="0">
-<segment>
-<pinref part="C3" gate="G$1" pin="2"/>
-<pinref part="R2" gate="G$1" pin="2"/>
-</segment>
-</net>
-<net name="N$4" class="0">
-<segment>
-<pinref part="IC1" gate="G$1" pin="OUT"/>
-<pinref part="C1" gate="G$1" pin="+"/>
-<pinref part="C3" gate="G$1" pin="1"/>
-<wire x1="152.4" y1="182.88" x2="172.72" y2="182.88" width="0.1524" layer="91"/>
-<wire x1="172.72" y1="182.88" x2="182.88" y2="182.88" width="0.1524" layer="91"/>
-<wire x1="172.72" y1="180.34" x2="172.72" y2="182.88" width="0.1524" layer="91"/>
-<junction x="172.72" y="182.88"/>
-</segment>
-</net>
-<net name="N$6" class="0">
-<segment>
-<pinref part="IC1" gate="G$1" pin="GAIN@1"/>
-<wire x1="144.78" y1="187.96" x2="144.78" y2="185.42" width="0.1524" layer="91"/>
-</segment>
-</net>
-<net name="N$7" class="0">
-<segment>
-<pinref part="C1" gate="G$1" pin="-"/>
-<pinref part="SPK" gate="G$1" pin="1"/>
-<wire x1="190.5" y1="182.88" x2="251.46" y2="182.88" width="0.1524" layer="91"/>
-</segment>
-</net>
 <net name="N$9" class="0">
 <segment>
@@
 <pinref part="IC2" gate="B" pin="OUT"/>
 <wire x1="154.94" y1="48.26" x2="149.86" y2="48.26" width="0.1524" layer="91"/>
-</segment>
-</net>
-<net name="N$5" class="0">
-<segment>
-<pinref part="C2" gate="G$1" pin="2"/>
-<pinref part="IC1" gate="G$1" pin="+IN"/>
-<wire x1="116.84" y1="185.42" x2="134.62" y2="185.42" width="0.1524" layer="91"/>
 </segment>
 </net>
@@
 </segment>
 </net>
+<net name="N$1" class="0">
+<segment>
+<pinref part="IC3" gate="1" pin="W"/>
+<wire x1="71.12" y1="170.18" x2="66.04" y2="170.18" width="0.1524" layer="91"/>
+</segment>
+</net>

Commit message: This should work…
Parts:
- removed C8: 2.2nF, rcl:C-US025-025X050
- removed SPK1: (no value), pinhead:PINHD-1X2
- added R10: 10K, resistor:R-US_0207/10
- added TOUCH: (no value), adafruit:PINHD-1X1
- C2: value 0.01u -> 2.2
- C3: value 0.047u -> 2.2
- C5: value 100uF -> 1; device rcl:CPOL-EUE2.5-5 -> rcl:C-US025-025X050
- C6: value 10nF -> 2.2nF
- C7: value 1 -> 10nF
- IC3: value DS1804 -> DS1804-10k
- R2: value 10 -> 8k
- R3: value 10K -> 10k
- R4: value 100K -> 15K
- R6: value 15K -> 33K
- R9: value 33K -> 100K
Connections:
- new net N$2: C2.1, IN.2
- new net N$3: C2.2, R3.2
- new net N$4: R2.2, R3.1, U2.IN-
- new net N$5: C3.1, U2.BYPASS, U2.IN+
- new net N$6: SPK.1, U2.VOUTB
- new net N$7: IC3.L, IC3.W, R2.1
- new net VCC: CTRL.8, U2.SHDN
- net +5V: now also C1.+, IC3.VCC, R10.2, U2.V+; no longer R3.2
- net GND: now also C1.-, C3.2, C5.2, C6.2, IC3.GND, R9.1, U2.V-; no longer C7.2, C8.2, R6.1, SPK.2
- net N$1: now also IC3.H, SPK.2, U2.VOUTA; no longer IC3.W
- net N$11: now also R6.2; no longer R9.2
- net N$12: now also R4.2; no longer R6.2
- net N$13: now also C6.1, R6.1; no longer C8.1, R9.1
- net N$15: now also C5.1, R9.2; no longer C7.1, R4.2
- net N$16: now also C7.1; no longer C6.1
- net N$17: now also C7.2; no longer C6.2
- net N$22: now also TOUCH.1; no longer SPK1.1
- net N$9: now also R10.1; no longer R3.1
Other:
- moved on the sheet: C1, C2, C3, C6, C7, IC3, IN, R1, R2, R3, R4, R6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

Commit message: Waiting for proto board test design
Parts:
- added C8: 0.1, rcl:C-US025-025X050
- C4: value 0.1 -> 1
- C7: value 10nF -> 0.01
- R10: value 10K -> 1k
Connections:
- net +5V: now also C8.1
- net GND: now also C8.2
- net N$10: no longer IC4.H
- net N$7: no longer IC3.L
Changed lines of the file:
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@@
 <part name="IC4" library="pot-xicor" deviceset="X9C102*" device="P" value="DS1804"/>
 <part name="R2" library="resistor" deviceset="R-US_" device="0207/10" value="8k"/>
-<part name="R10" library="resistor" deviceset="R-US_" device="0207/10" value="10K"/>
+<part name="R10" library="resistor" deviceset="R-US_" device="0207/10" value="1k"/>
 <part name="R9" library="resistor" deviceset="R-US_" device="0207/10" value="100K"/>
 <part name="R5" library="resistor" deviceset="R-US_" device="0207/10" value="10K"/>
@@
 <part name="C1" library="rcl" deviceset="CPOL-EU" device="E2-5" value="250u"/>
 <part name="C3" library="rcl" deviceset="C-US" device="025-025X050" value="2.2"/>
-<part name="C4" library="rcl" deviceset="C-US" device="025-025X050" value="0.1"/>
+<part name="C4" library="rcl" deviceset="C-US" device="025-025X050" value="1"/>
 <part name="SUPPLY4" library="supply2" deviceset="+5V" device=""/>
 <part name="SUPPLY5" library="supply2" deviceset="GND" device=""/>
@@
 <part name="U1" library="SparkFun-DigitalIC" deviceset="AT42QT1010" device="SOT23"/>
 <part name="R1" library="resistor" deviceset="R-US_" device="0207/10" value="10k"/>
-<part name="C7" library="rcl" deviceset="C-US" device="025-025X050" value="10nF"/>
+<part name="C7" library="rcl" deviceset="C-US" device="025-025X050" value="0.01"/>
 <part name="R8" library="resistor" deviceset="R-US_" device="0207/10" value="100K"/>
 <part name="C5" library="rcl" deviceset="C-US" device="025-025X050" value="1"/>
@@
 <part name="SUPPLY14" library="supply2" deviceset="GND" device=""/>
 <part name="TOUCH" library="adafruit" deviceset="PINHD-1X1" device=""/>
+<part name="C8" library="rcl" deviceset="C-US" device="025-025X050" value="0.1"/>
 </parts>
 <sheets>
@@
 <instance part="SUPPLY14" gate="GND" x="170.18" y="157.48"/>
 <instance part="TOUCH" gate="G$1" x="259.08" y="73.66" rot="R180"/>
+<instance part="C8" gate="G$1" x="167.64" y="68.58"/>
 </instances>
 <busses>
@@
 <segment>
 <pinref part="U1" gate="G$1" pin="VSS"/>
-<wire x1="177.8" y1="63.5" x2="177.8" y2="48.26" width="0.1524" layer="91"/>
+<wire x1="177.8" y1="63.5" x2="177.8" y2="55.88" width="0.1524" layer="91"/>
 <pinref part="SUPPLY13" gate="GND" pin="GND"/>
+<pinref part="C8" gate="G$1" pin="2"/>
+<wire x1="177.8" y1="55.88" x2="177.8" y2="48.26" width="0.1524" layer="91"/>
+<wire x1="177.8" y1="55.88" x2="167.64" y2="55.88" width="0.1524" layer="91"/>
+<wire x1="167.64" y1="55.88" x2="167.64" y2="63.5" width="0.1524" layer="91"/>
+<junction x="177.8" y="55.88"/>
 </segment>
 <segment>
@@
 <wire x1="218.44" y1="86.36" x2="195.58" y2="86.36" width="0.1524" layer="91"/>
 <junction x="195.58" y="86.36"/>
+<pinref part="C8" gate="G$1" pin="1"/>
+<wire x1="195.58" y1="86.36" x2="167.64" y2="86.36" width="0.1524" layer="91"/>
+<wire x1="167.64" y1="86.36" x2="167.64" y2="71.12" width="0.1524" layer="91"/>
 </segment>
 <segment>
@@
 <wire x1="71.12" y1="83.82" x2="71.12" y2="48.26" width="0.1524" layer="91"/>
 <junction x="71.12" y="48.26"/>
-<pinref part="IC4" gate="1" pin="H"/>
-<wire x1="78.74" y1="88.9" x2="71.12" y2="88.9" width="0.1524" layer="91"/>
-<wire x1="71.12" y1="88.9" x2="71.12" y2="83.82" width="0.1524" layer="91"/>
-<junction x="71.12" y="83.82"/>
 </segment>
 </net>
@@
 <pinref part="IC3" gate="1" pin="W"/>
 <pinref part="R2" gate="G$1" pin="1"/>
-<wire x1="137.16" y1="172.72" x2="134.62" y2="172.72" width="0.1524" layer="91"/>
-<pinref part="IC3" gate="1" pin="L"/>
-<wire x1="134.62" y1="172.72" x2="132.08" y2="172.72" width="0.1524" layer="91"/>
-<wire x1="137.16" y1="167.64" x2="134.62" y2="167.64" width="0.1524" layer="91"/>
-<wire x1="134.62" y1="167.64" x2="134.62" y2="172.72" width="0.1524" layer="91"/>
-<junction x="134.62" y="172.72"/>
-</segment>
-</net>
+<wire x1="137.16" y1="172.72" x2="132.08" y2="172.72" width="0.1524" layer="91"/>
+</segment>
+</net>

Commit message: Final beta
Parts:
- removed C7: 0.01, rcl:C-US025-025X050
- removed C8: 0.1, rcl:C-US025-025X050
- removed R1: 10k, resistor:R-US_0207/10
- removed U1: AT42QT1010SOT23, SparkFun-DigitalIC:AT42QT1010SOT23
- R4: value 15K -> 15k
- R5: value 10K -> 10k
- R6: value 33K -> 33k
- R7: value 1K -> 1k
- R8, R9: value 100K -> 100k
- TOUCH: device adafruit:PINHD-1X1 -> adafruit:PINHD-1X3
Connections:
- removed net N$16: C7.1, R1.2, U1.SNSK
- removed net N$17: C7.2, U1.SNS
- removed net N$24: CTRL.6, U1.OUT
- net +5V: now also TOUCH.2; no longer C8.1, U1.SYNC/MODE, U1.VDD
- net GND: now also TOUCH.3; no longer C8.2, U1.VSS
- net N$22: now also CTRL.6; no longer R1.1
Other:
- note added: "A"
- moved on the sheet: CTRL

Commit message: Minor stuffs
Parts:
- removed R2: 8k, resistor:R-US_0207/10
- IC3: value DS1804-10k -> DS1804-50k
- IC4: value DS1804 -> DS1804-100k
- R3: value 10k -> 20k
Connections:
- removed net N$7: IC3.W, R2.1
- net N$4: now also IC3.W; no longer R2.2
Changed lines of the file:
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@@
 <part name="FRAME1" library="frames" deviceset="FRAME_A_L" device=""/>
 <part name="IC2" library="linear" deviceset="TL084" device="P"/>
-<part name="IC3" library="pot-xicor" deviceset="X9C102*" device="P" value="DS1804-10k"/>
-<part name="IC4" library="pot-xicor" deviceset="X9C102*" device="P" value="DS1804"/>
-<part name="R2" library="resistor" deviceset="R-US_" device="0207/10" value="8k"/>
+<part name="IC3" library="pot-xicor" deviceset="X9C102*" device="P" value="DS1804-50k"/>
+<part name="IC4" library="pot-xicor" deviceset="X9C102*" device="P" value="DS1804-100k"/>
 <part name="R10" library="resistor" deviceset="R-US_" device="0207/10" value="1k"/>
 <part name="R9" library="resistor" deviceset="R-US_" device="0207/10" value="100k"/>
@@
 <part name="C6" library="rcl" deviceset="C-US" device="025-025X050" value="2.2nF"/>
 <part name="U2" library="Analog Devices_By_element14_Batch_1" deviceset="SSM2211SZ" device=""/>
-<part name="R3" library="resistor" deviceset="R-US_" device="0207/10" value="10k"/>
+<part name="R3" library="resistor" deviceset="R-US_" device="0207/10" value="20k"/>
 <part name="SUPPLY3" library="supply2" deviceset="VCC" device="" value="Enabled"/>
 <part name="SUPPLY6" library="supply2" deviceset="VCC" device="" value="Enabled"/>
@@
 <instance part="IC3" gate="1" x="149.86" y="172.72" rot="MR0"/>
 <instance part="IC4" gate="1" x="91.44" y="83.82" rot="MR0"/>
-<instance part="R2" gate="G$1" x="127" y="172.72" rot="R180"/>
 <instance part="R10" gate="G$1" x="33.02" y="60.96" rot="R90"/>
 <instance part="R9" gate="G$1" x="58.42" y="38.1" rot="R90"/>
@@
 <wire x1="68.58" y1="144.78" x2="116.84" y2="144.78" width="0.1524" layer="91"/>
 <wire x1="116.84" y1="144.78" x2="116.84" y2="172.72" width="0.1524" layer="91"/>
-<pinref part="R2" gate="G$1" pin="2"/>
-<wire x1="116.84" y1="172.72" x2="121.92" y2="172.72" width="0.1524" layer="91"/>
 <junction x="68.58" y="162.56"/>
+<pinref part="IC3" gate="1" pin="W"/>
+<wire x1="137.16" y1="172.72" x2="134.62" y2="172.72" width="0.1524" layer="91"/>
+<wire x1="134.62" y1="172.72" x2="132.08" y2="172.72" width="0.1524" layer="91"/>
+<wire x1="116.84" y1="172.72" x2="132.08" y2="172.72" width="0.1524" layer="91"/>
 </segment>
 </net>
@@
 </segment>
 </net>
-<net name="N$7" class="0">
-<segment>
-<pinref part="IC3" gate="1" pin="W"/>
-<pinref part="R2" gate="G$1" pin="1"/>
-<wire x1="137.16" y1="172.72" x2="132.08" y2="172.72" width="0.1524" layer="91"/>
-</segment>
-</net>

Commit message: Final version
Parts:
- added D1: 1N5817, adafruit:SCHOTTKY-DIODEDO41-7
- added R1: 2k, rcl:R-US_0204/2V
- added R11: 100k, rcl:R-US_0204/2V
- added R12: 15k, rcl:R-US_0204/2V
- added R13: 5.1k, rcl:R-US_0204/2V
- added R14: 20k, rcl:R-US_0204/2V
- added R2: 1k, rcl:R-US_0204/2V
- C1: value 250u -> 250; device rcl:CPOL-EUE2-5 -> rcl:CPOL-USE3.5-10
- C2, C3: device rcl:C-US025-025X050 -> rcl:CPOL-USE3.5-8
- C4, C5: device rcl:C-US025-025X050 -> rcl:CPOL-USE2-4
- C6: value 2.2nF -> 10; device rcl:C-US025-025X050 -> rcl:CPOL-USE2-4
- IC4: value DS1804-100k -> DS1804-10k
- R10: device resistor:R-US_0207/10 -> rcl:R-US_0204/2V
- R3: value 20k -> 100k; device resistor:R-US_0207/10 -> rcl:R-US_0204/2V
- R4: value 15k -> 100k; device resistor:R-US_0207/10 -> rcl:R-US_0204/2V
- R5: value 10k -> 1M; device resistor:R-US_0207/10 -> rcl:R-US_0204/2V
- R6: value 33k -> 10k; device resistor:R-US_0207/10 -> rcl:R-US_0204/2V
- R7: value 1k -> 100; device resistor:R-US_0207/10 -> rcl:R-US_0204/2V
- R8: value 100k -> 10k; device resistor:R-US_0207/10 -> rcl:R-US_0204/2V
- R9: value 100k -> 1k; device resistor:R-US_0207/10 -> rcl:R-US_0204/2V
- renumbered IN to LINE-IN, U2 to IC1
Connections:
- removed net N$14: CTRL.9, IC2B.OUT
- new net N$17: D1.A, IC2B.OUT
- new net N$23: D1.C, IC2B.+IN, R7.1
- new net N$24: C6.+, IC2C.+IN, R7.2, R8.2
- new net N$25: IC2C.-IN, R9.1
- new net N$26: IC2C.OUT, R10.1, R9.2
- new net N$27: IC2D.+IN, R10.2, R11.1
- new net N$28: CTRL.9, IC2D.OUT, R11.2
- new net N$29: IC2D.-IN, R12.2, R13.1
- new net N$7: IC4.L, R13.2
- net +5V: now also IC4.H, IC4.W, R1.2, R3.2; no longer R10.2, R5.2, R8.2
- net GND: now also C3.-, C6.-, R12.1, R8.1; no longer C3.2, C5.2, C6.2, R9.1
- net N$10: now also R2.2, R5.1; no longer IC4.W, R7.1
- net N$11: now also C5.+, R5.2; no longer IC4.L, R6.2
- net N$12: now also C5.-, R6.1; no longer IC2B.-IN, R4.2, R5.1
- net N$13: now also IC2B.-IN, R6.2; no longer C6.1, IC2B.+IN, R6.1
- net N$15: now also R3.1, R4.2; no longer C5.1, R8.1, R9.2
- net N$2: now also C2.+; no longer C2.1
- net N$3: now also C2.-, R14.1; no longer C2.2, R3.2
- net N$4: now also IC3.L, R14.2; no longer R3.1
- net N$5: now also C3.+; no longer C3.1
- net N$8: now also C4.-, R2.1; no longer C4.2, R7.2
- net N$9: now also C4.+, R1.1; no longer C4.1, R10.1
Other:
- moved on the sheet: CTRL, IC2A, IC2B, IC4, MIC, R10, R3, R4, R5, R6, R7, R8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
